Commit message: modify go2 urdf for choreonoid

File: genesis/assets/urdf/go2/urdf/go2.urdf (robot description, URDF)
Before this commit: robot go2_description, 29 links, 28 joints
Links:
- removed link Head_lower
- removed link Head_upper
- link imu: mass 0 -> 0.01
- link radar: mass 0 -> 0.01
Joints:
- removed joint Head_lower_joint
- removed joint Head_upper_joint

Commit message: use the same model between visual and collision of the calf links

File: genesis/assets/urdf/go2/urdf/go2.urdf (robot description, URDF)
Before this commit: robot go2_description, 27 links, 26 joints
Links:
- link FL_calf: geometry collision mesh filename=../dae/calf.dae; visual mesh filename=../dae/calf.dae
- link FR_calf: geometry collision mesh filename=../dae/calf_mirror.dae; visual mesh filename=../dae/calf_mirror.dae
- link RL_calf: geometry collision mesh filename=../dae/calf.dae; visual mesh filename=../dae/calf.dae
- link RR_calf: geometry collision mesh filename=../dae/calf_mirror.dae; visual mesh filename=../dae/calf_mirror.dae

Commit message: change weight of go2

File: genesis/assets/urdf/go2/urdf/go2.urdf (robot description, URDF)
Before this commit: robot go2_description, 27 links, 26 joints
Links:
- link FL_calf: mass 0.154 -> 0.231000
- link FL_foot: mass 0.04 -> 0.060000
- link FL_hip: mass 0.678 -> 1.017000
- link FL_thigh: mass 1.152 -> 1.728000
- link FR_calf: mass 0.154 -> 0.231000
- link FR_foot: mass 0.04 -> 0.060000
- link FR_hip: mass 0.678 -> 1.017000
- link FR_thigh: mass 1.152 -> 1.728000
- link RL_calf: mass 0.154 -> 0.231000
- link RL_foot: mass 0.04 -> 0.060000
- link RL_hip: mass 0.678 -> 1.017000
- link RL_thigh: mass 1.152 -> 1.728000
- link RR_calf: mass 0.154 -> 0.231000
- link RR_foot: mass 0.04 -> 0.060000
- link RR_hip: mass 0.678 -> 1.017000
- link RR_thigh: mass 1.152 -> 1.728000
- link base: mass 6.921 -> 10.381500
- link imu: mass 0.01 -> 0.015000
- link radar: mass 0.01 -> 0.015000
